File: kicad_pcb_model/wavplayer-1_2.kicad_pcb (KiCad board)
At the start: 2 copper layers, 27.5 x 67.2 mm, 14 parts, among them SW1 DOWN, SW2 BACK, SW3 UP, SW4 ENTER

Commit message: fixed pins not being set correctly
Parts:
- moved ESP1 17.8 mm to (126.0, 116.2), turned to 90 degrees
Connections:
- ESP1 pad 4: /SDA -> /SCL
- ESP1 pad 5: /SCL -> /SDA
Routing:
- net /MISO: track 11.6 -> 25.6 mm
- net /CS: track 11.0 -> 21.2 mm
- net /MOSI: track 11.0 -> 17.4 mm
Changed lines of the file:
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@@
 	(footprint "Connector_PinHeader_2.54mm:PinHeader_1x08_P2.54mm_Vertical"
 		(layer "F.Cu")
-		(at 143.74 116.25 -90)
+		(at 125.96 116.25 90)
 		(descr "Through hole straight pin header, 1x08, 2.54mm pitch, single row")
 		(tags "Through hole pin header THT 1x08 2.54mm single row")
@@
 		(duplicate_pad_numbers_are_jumpers no)
 		(fp_line
+			(start -1.38 -1.38)
+			(end 0 -1.38)
+			(stroke
+				(width 0.12)
+				(type solid)
+			)
+			(layer "F.SilkS")
+		)
+		(fp_line
+			(start -1.38 0)
+			(end -1.38 -1.38)
+			(stroke
+				(width 0.12)
+				(type solid)
+			)
+			(layer "F.SilkS")
+		)
+		(fp_line
+			(start 1.38 1.27)
+			(end 1.38 19.16)
+			(stroke
+				(width 0.12)
+				(type solid)
+			)
+			(layer "F.SilkS")
+		)
+		(fp_line
+			(start -1.38 1.27)
+			(end 1.38 1.27)
+			(stroke
+				(width 0.12)
+				(type solid)
+			)
+			(layer "F.SilkS")
+		)
+		(fp_line
+			(start -1.38 1.27)
+			(end -1.38 19.16)
+			(stroke
+				(width 0.12)
+				(type solid)
+			)
+			(layer "F.SilkS")
+		)
+		(fp_line
 			(start -1.38 19.16)
 			(end 1.38 19.16)
-			(stroke
-				(width 0.12)
-				(type solid)
-			)
-			(layer "F.SilkS")
-		)
-		(fp_line
-			(start -1.38 1.27)
-			(end -1.38 19.16)
-			(stroke
-				(width 0.12)
-				(type solid)
-			)
-			(layer "F.SilkS")
-		)
-		(fp_line
-			(start -1.38 1.27)
-			(end 1.38 1.27)
-			(stroke
-				(width 0.12)
-				(type solid)
-			)
-			(layer "F.SilkS")
-		)
-		(fp_line
-			(start 1.38 1.27)
-			(end 1.38 19.16)
-			(stroke
-				(width 0.12)
-				(type solid)
-			)
-			(layer "F.SilkS")
-		)
-		(fp_line
-			(start -1.38 0)
-			(end -1.38 -1.38)
-			(stroke
-				(width 0.12)
-				(type solid)
-			)
-			(layer "F.SilkS")
-		)
-		(fp_line
-			(start -1.38 -1.38)
-			(end 0 -1.38)
 			(stroke
 				(width 0.12)
@@
 		)
 		(fp_line
+			(start 1.27 -1.27)
+			(end 1.27 19.05)
+			(stroke
+				(width 0.1)
+				(type solid)
+			)
+			(layer "F.Fab")
+		)
+		(fp_line
+			(start -0.635 -1.27)
+			(end 1.27 -1.27)
+			(stroke
+				(width 0.1)
+				(type solid)
+			)
+			(layer "F.Fab")
+		)
+		(fp_line
+			(start -1.27 -0.635)
+			(end -0.635 -1.27)
+			(stroke
+				(width 0.1)
+				(type solid)
+			)
+			(layer "F.Fab")
+		)
+		(fp_line
+			(start 1.27 19.05)
+			(end -1.27 19.05)
+			(stroke
+				(width 0.1)
+				(type solid)
+			)
+			(layer "F.Fab")
+		)
+		(fp_line
 			(start -1.27 19.05)
 			(end -1.27 -0.635)
@@
 			(layer "F.Fab")
 		)
-		(fp_line
-			(start 1.27 19.05)
-			(end -1.27 19.05)
-			(stroke
-				(width 0.1)
-				(type solid)
-			)
-			(layer "F.Fab")
-		)
-		(fp_line
-			(start -1.27 -0.635)
-			(end -0.635 -1.27)
-			(stroke
-				(width 0.1)
-				(type solid)
-			)
-			(layer "F.Fab")
-		)
-		(fp_line
-			(start -0.635 -1.27)
-			(end 1.27 -1.27)
-			(stroke
-				(width 0.1)
-				(type solid)
-			)
-			(layer "F.Fab")
-		)
-		(fp_line
-			(start 1.27 -1.27)
-			(end 1.27 19.05)
-			(stroke
-				(width 0.1)
-				(type solid)
-			)
-			(layer "F.Fab")
-		)
 		(fp_text user "${REFERENCE}"
 			(at -2.75 9.24 0)
@@
 		)
 		(pad "1" thru_hole rect
-			(at 0 0 270)
+			(at 0 0 90)
 			(size 1.7 1.7)
 			(drill 1)
@@
 		)
 		(pad "2" thru_hole circle
-			(at 0 2.54 270)
+			(at 0 2.54 90)
 			(size 1.7 1.7)
 			(drill 1)
@@
 		)
 		(pad "3" thru_hole circle
-			(at 0 5.08 270)
+			(at 0 5.08 90)
 			(size 1.7 1.7)
 			(drill 1)
@@
 		)
 		(pad "4" thru_hole circle
-			(at 0 7.62 270)
+			(at 0 7.62 90)
+			(size 1.7 1.7)
+			(drill 1)
+			(layers "*.Cu" "*.Mask")
+			(remove_unused_layers no)
+			(net "/SCL")
+			(pinfunction "Pin_4_4")
+			(pintype "passive")
+		)
+		(pad "5" thru_hole circle
+			(at 0 10.16 90)
 			(size 1.7 1.7)
 			(drill 1)
@@
 			(remove_unused_layers no)
 			(net "/SDA")
-			(pinfunction "Pin_4_4")
-			(pintype "passive")
-		)
-		(pad "5" thru_hole circle
-			(at 0 10.16 270)
-			(size 1.7 1.7)
-			(drill 1)
-			(layers "*.Cu" "*.Mask")
-			(remove_unused_layers no)
-			(net "/SCL")
 			(pinfunction "Pin_5_5")
 			(pintype "passive")
 		)
 		(pad "6" thru_hole circle
-			(at 0 12.7 270)
+			(at 0 12.7 90)
 			(size 1.7 1.7)
 			(drill 1)
@@
 		)
 		(pad "7" thru_hole circle
-			(at 0 15.24 270)
+			(at 0 15.24 90)
 			(size 1.7 1.7)
 			(drill 1)
@@
 		)
 		(pad "8" thru_hole circle
-			(at 0 17.78 270)
+			(at 0 17.78 90)
 			(size 1.7 1.7)
 			(drill 1)
@@
 	)
 	(gr_text "PCM5102A BCK  GPIO1 ACD1_1    (1) Sch T2\n\nPCM5102A LRCK GPIO2 ACD1_2    (2) Sch T3\n\nPCM5102A DATA GPIO3 ACD1_3    (3) Sch T4\n\nPCM5102A 3.3V 3.3V\n\nPCM5102A GND  GND\n\nSD       SCK  GPIO4 A4 / SCK  (4) Sch T5\n\nSD       MISO GPIO5 A5 / MISO (21) Sch B1\n\nSD       MOSI GPIO6 MOSI      (20) Sch B2\n\nSD       CS   GPIO7 SS/CS     (10) Sch B3\n\nSSD1306  SDA  GPIO8 SDA       (9) Sch B4\n\nSSD1306  SCL  GPIO9 SCL       (8) Sch B5\n"
-		(at 128 73.75 0)
+		(at 106 68.5 0)
 		(layer "Cmts.User")
 		(effects
@@
 	)
 	(segment
-		(start 136.12 116.25)
-		(end 137.67 117.8)
+		(start 137.67 117.8)
+		(end 136.12 116.25)
 		(width 0.2)
 		(layer "B.Cu")
@@
 	)
 	(segment
-		(start 143.74 116.25)
-		(end 143.74 107.47)
+		(start 143.153654 107.47)
+		(end 134.73 115.893654)
+		(width 0.2)
+		(layer "B.Cu")
+		(net "/MISO")
+	)
+	(segment
+		(start 134.056346 117.4)
+		(end 127.11 117.4)
+		(width 0.2)
+		(layer "B.Cu")
+		(net "/MISO")
+	)
+	(segment
+		(start 134.73 116.726346)
+		(end 134.056346 117.4)
 		(width 0.2)
 		(layer "B.Cu")
@@
 	)
 	(segment
-		(start 141.2 116.25)
-		(end 141.2 106.07)
-		(width 0.2)
-		(layer "B.Cu")
+		(start 127.11 117.4)
+		(end 125.96 116.25)
+		(width 0.2)
+		(layer "B.Cu")
+		(net "/MISO")
+	)
+	(segment
+		(start 134.73 115.893654)
+		(end 134.73 116.726346)
+		(width 0.2)
+		(layer "B.Cu")
+		(net "/MISO")
+	)
+	(segment
+		(start 143.74 107.47)
+		(end 143.153654 107.47)
+		(width 0.2)
+		(layer "B.Cu")
+		(net "/MISO")
+	)
+	(segment
+		(start 140.63 105.5)
+		(end 139.48 106.65)
+		(width 0.2)
+		(layer "F.Cu")
+		(net "/MOSI")
+	)
+	(segment
+		(start 138.1 106.65)
+		(end 128.5 116.25)
+		(width 0.2)
+		(layer "F.Cu")
+		(net "/MOSI")
+	)
+	(segment
+		(start 139.48 106.65)
+		(end 138.1 106.65)
+		(width 0.2)
+		(layer "F.Cu")
 		(net "/MOSI")
 	)
@@
 	)
 	(segment
-		(start 138.66 116.25)
-		(end 138.66 106.07)
-		(width 0.2)
-		(layer "B.Cu")
+		(start 129.89 117.4)
+		(end 128.023654 117.4)
+		(width 0.2)
+		(layer "F.Cu")
 		(net "/CS")
 	)
+	(segment
+		(start 127.35 115.773654)
+		(end 137.623654 105.5)
+		(width 0.2)
+		(layer "F.Cu")
+		(net "/CS")
+	)
+	(segment
+		(start 127.35 116.726346)
+		(end 127.35 115.773654)
+		(width 0.2)
+		(layer "F.Cu")
+		(net "/CS")
+	)
+	(segment
+		(start 131.04 116.25)
+		(end 129.89 117.4)
+		(width 0.2)
+		(layer "F.Cu")
+		(net "/CS")
+	)
+	(segment
+		(start 137.623654 105.5)
+		(end 138.09 105.5)
+		(width 0.2)
+		(layer "F.Cu")
+		(net "/CS")
+	)
+	(segment
+		(start 128.023654 117.4)
+		(end 127.35 116.726346)
+		(width 0.2)
+		(layer "F.Cu")
+		(net "/CS")
+	)
